Commit message: fix(urdf): align gripper_frame_link with actual fingertip (98mm → 85mm)
URDF의 gripper_frame_link가 모터 회전축에서 98.4mm 앞에 정의돼 있었으나,
실측한 fingertip 위치는 85mm 앞 → 13mm 차이로 인해 IK가 grasp 시 잘못된
EE 위치를 명령했던 문제 해결.

원인:
  - gripper_frame_joint origin xyz="-0.0079 -0.000218121 -0.0981274"
    → gripper_link 에서 98.4mm 앞 (URDF 가정)
  - 실제 fingertip 은 모터 회전축에서 85mm 앞 (자로 측정)
  - 13.6mm 차이 → 로봇 좌표계 IK target 이 실제 grasp 위치와 어긋남

증상:
  - VLM 으로 검출한 객체 중심을 잡으려 할 때, 그리퍼 TIP 이 객체 중앙에서
    앞쪽으로 쏠려 미끄러짐 ("ee가 물건의 정중앙을 잡지 못하고 좀 더 앞쪽")
  - skills_lerobot.py 의 pitch compensation (drift only) 으로는 부분적으로만
    해결되어 grasp 정확도 저하

해결:
  - gripper_frame_joint origin 을 동일 방향, 짧은 거리로 변경:
    xyz="-0.006824 -0.000189 -0.084754" (= 85mm 거리, 동일 단위벡터)
  - 결과: gripper_frame_link 가 이제 fingertip 자체를 가리킴
  - FK/IK 가 자동으로 fingertip 기준 동작 → 별도 보정 불필요
  - skills/skills_lerobot.py 의 GRIPPER_TIP_LENGTH 보정 로직 제거
    (execute_pick_object, execute_place_object 두 곳)

영향:
  - SO-101 robot 6대 (robot0/1/2/3/6/8) URDF 모두 동일 수정
  - 기존 Charuco extrinsics 캘리브 데이터는 무효화 (gripper_frame_link 위치
    13.6mm 변경됨) → 재캘리브 필요
  - max_reach 가 13.6mm 짧아짐 (kinematics 자동 재계산)
  - 시뮬레이션/시각화 정확도 향상 (URDF 가 실 물리 위치 반영)

검증:
  - 한 객체를 두 다른 높이 (테이블 / 책 4cm 위) 에서 검출 → xy 차이 2mm 이내
    (이전 단일 평면 캘리브 8.4mm → 다중 높이 캘리브 2mm 까지 개선됨)
  - 잔여 grasp 오차의 원인이 시차 (A) 가 아닌 그리퍼 형상 (F) 임을 확인,
    URDF 수정으로 F 근본 해결

Co-Authored-By: Claude Opus 4.7 (1M context) <noreply@anthropic.com>

File: assets/urdf/so101_robot0.urdf (robot description, URDF)
Before this commit: robot so101_new_calib, 8 links, 7 joints
Joints:
- joint gripper_frame_joint: origin xyz=-0.0079 -0.000218121 -0.0981274 rpy=0 3.14159 0 -> xyz=-0.006824 -0.000189 -0.084754 rpy=0 3.14159 0

File: assets/urdf/so101_robot1.urdf (robot description, URDF)
Before this commit: robot so101_new_calib, 8 links, 7 joints
Joints:
- joint gripper_frame_joint: origin xyz=-0.0079 -0.000218121 -0.0981274 rpy=0 3.14159 0 -> xyz=-0.006824 -0.000189 -0.084754 rpy=0 3.14159 0
