Commit message: fix: subgoal poisson-disk 선택 + gripper limit/material 패치
subgoal_selector
- 후보 선택을 argmax(gain) 에서 poisson-disk 로 교체. 최소 분리거리
  r_min = 0.75 * scale 를 만족하는 후보를 무작위 채택하고, 없으면 gain
  순으로 폴백한다.
- r_min 을 descriptor 공간에서 계산하도록 수정. 이전에는 offset 공간의
  R=0.05 를 descriptor 공간의 분리거리와 비교해 통과 후보가 1개로 줄고
  선택이 사실상 argmax 로 축퇴했다 (실측: 67회 중 63회 argmax 와 동일).

terminal_descriptor
- terminal region 기술자 계산 보완 (분리거리 산출에 사용).

assets/urdf/so101_robot3.urdf
- gripper joint lower limit -0.00153 -> -0.18 rad. ADC 의 normalized=0 이
  RWDC normalized=-100 과 같은 엔코더 위치이고 그것이 -0.18 rad 이다.
  이 값이 없으면 SCRAPE 경로에서 gym.make 가 범위 검사로 죽는다.
- wrist_roll / moving_jaw material 을 3d_printed -> sts3215 로 교정.
  렌더링·데이터셋에서 그리퍼가 노란색으로 나오던 문제.

File: assets/urdf/so101_robot3.urdf (robot description, URDF)
Before this commit: robot so101_new_calib, 8 links, 7 joints
Joints:
- joint gripper: limit lower=-0.00153 upper=2.25648 effort=10 velocity=10 -> lower=-0.18 upper=2.25648 effort=10 velocity=10
